File: eda-logical/logical.kicad_pcb (KiCad board)
At the start: 2 copper layers, 189.7 x 124 mm, 42 parts, among them P1 IO_PLUG_M22, Q101 2N1305, Q102 2N1304, Q103 2N1038, Q104 2N1038, Q105 2N697, Q106 2N697, Q107 2N697

Commit message: minor cleanups and tweaks
Parts:
- R103, R104: value 2K -> 2000
- R111: value 1.5K -> 1500
- R124: value 1.6K -> 1600
- R125: value 0.1 ? -> 0.1?
Changed lines of the file:
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@@
 			)
 		)
-		(property "Value" "0.1 ?"
+		(property "Value" "0.1?"
 			(at 12.7 1.5 0)
 			(layer "F.Fab")
@@
 			)
 		)
+		(property "Field5" "Vf=0.7V"
+			(at 0 0 180)
+			(unlocked yes)
+			(layer "F.Fab")
+			(hide yes)
+			(effects
+				(font
+					(size 1 1)
+					(thickness 0.15)
+				)
+			)
+		)
 		(property ki_fp_filters "TO-???* *_Diode_* *SingleDiode* D_*")
 		(sheetname "Root")
@@
 			)
 		)
-		(property "Value" "2K"
+		(property "Value" "2000"
 			(at 12.7 1.5 0)
 			(layer "F.Fab")
@@
 			)
 		)
-		(property "Field5" "Vz=9.2V"
+		(property "Field5" "Vz=9.4V"
 			(at 0 0 0)
 			(unlocked yes)
@@
 			)
 		)
-		(property "Value" "2K"
+		(property "Value" "2000"
 			(at 12.7 -1.5 0)
 			(layer "F.Fab")
@@
 			)
 		)
-		(property "Value" "1.5K"
+		(property "Value" "1500"
 			(at 12.7 1.5 0)
 			(layer "F.Fab")
@@
 			)
 		)
-		(property "Value" "1.6K"
+		(property "Value" "1600"
 			(at 12.7 3.370001 0)
 			(layer "F.Fab")
@@
 					(thickness 0.15)
 				)
+			)
+		)
+		(property "Field5" "Vf=0.7V"
+			(at 0 0 180)
+			(unlocked yes)
+			(layer "F.Fab")
+			(hide yes)
+			(effects
+				(font
+					(size 1 1)
+					(thickness 0.15)
+				)
