File: eda-logical/logical.kicad_sch (KiCad schematic)
At the start: 48 parts, among them J1 IO_JACK_F22, P1 IO_PLUG_M22, Q101 2N1305, Q102 2N1304, Q103 2N1038, Q104 2N1038, Q105 2N697, Q106 2N697, Q107 2N697

Commit message: minor cleanups and tweaks
Parts:
- added SW1: SW_SPST, symbol Switch:SW_SPST
- CR105, CR106: Field5 (none) -> Vf=0.7V
- CR108: Field5 Vz=9.2V -> Vz=9.4V
- R103, R104: value 2K -> 2000
- R111: value 1.5K -> 1500
- R124: value 1.6K -> 1600
- R125: value 0.1 ? -> 0.1?
Connections:
- net -VDC: now also SW1.2 (B)
- net V25OUT-: now reaches J1.16 (Pin_6)
- net V25OUT+: now reaches J1.6 (Pin_6)
- net VCC_OUTPUT+ renamed VDC_OUT_DIFF+
- net VCC_OUTPUT- renamed VDC_OUT_DIFF-
Other:
- sheet Traced Circuit renamed TRACED CIRCUIT
- note added: "+24.4V DROP"
- note added: "+25.8V OUTPUT"
- note added: "+25.8V RETURN"
- note added: "+80.6V DROP"
- note added: "+9.4V DROP"
- note added: "500 OHM ADJUSTMENT"
- note added: "CURRENT Q107 BIASES AMP TRANSISTORS?"
- note added: "CURRENT SENSE TRIMMING CIRCUIT"
- note added: "DIFFERENTIAL AMPLIFIER"
- note added: "EDGE CONNECTOR"
- note added: "EXCITATION CIRCUIT PRECISION REF"
- note added: "FLOATING +25.8VDC SUPPLY"
- note added: "FLOATING PRECISION +9.4V DC REFERENCE?"
- note added: "FOR REFERENCE"
- note added: "IN+"
- note added: "IN-"
- note added: "INPUT"
- note added: "OUT+"
- note added: "OUT-"
- note added: "OUTPUT"
- note added: "OUTPUT DRIVE DISABLE?"
- note added: "Q101/Q102 FUNCTION: * 25.8V OUTPUT DRIVERS * CR101/CR102 BYPASS"
- note added: "SENSOR BRIDGE"
- note added: "SUPER ULTRA THERMALLY COMPENSATED"
- note added: "WHY ALL THIS ADJUSTMENT? GAIN AND OFFSET? BRIDGE RESISTORS?"
- note added: "ZENER REFERENCE"
- note removed: "+24.2V"
- note removed: "+9.2V DROP"
- note removed: "500 OHM ADNUSTMENT"
- note removed: "BEFORE ZENER CR101 BREAKDOWN, CURRENT FLOWS THROUGH Q101. THEN STOPS?"
- note removed: "FLOATING PRECISION +9.2V DC REFERENCE?"
- note removed: "INPUT CURRENT TO CONTROL OUTPUT CURRENT (RETURN PATH?)"
- note removed: "INPUT?"
- note removed: "NET1"
- note removed: "NET10"
- note removed: "NET11"
- note removed: "NET12"
- note removed: "NET13"
- note removed: "NET14"
- note removed: "NET15"
- note removed: "NET16"
- note removed: "NET17"
- note removed: "NET18"
- note removed: "NET19"
- note removed: "NET2"
- note removed: "NET20"
- note removed: "NET21"
- note removed: "NET3"
- note removed: "NET4"
- note removed: "NET5"
- note removed: "NET6"
- note removed: "NET7"
- note removed: "NET8"
- note removed: "NET9"
- note removed: "OUTPUT DRIVE ENABLE ?"
- note removed: "OUTPUT?"
- note removed: "SEE NOTE ABOVE @Q101"
- note removed: "SENSOR BRIDGE ???"
- note removed: "SUPER THERMALLY COMPENSATED"
- note removed: "WHAT'S ALL THIS ADHUSTMENT FOR ? COULD BE GAIN AND OFFSET ?"
- moved on the sheet: CR101, CR102, CR103, CR104, CR105, CR106, CR107, CR108, CR109, J1, P1, Q101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
